Commit message: Add Swift visualization and refine robot URDF structure
- Add cardboard.urdf for workspace visualization
- Implement Swift-based web viewer with proper URDF rendering
- Refactor robot.urdf with prismatic shoulder joint and L-shaped offset
- Add Swift compatibility patch for Python 3.12
- Update simulator with offset geometry visualization
- Adjust workspace positioning and joint limits for improved reachability

File: config/robot copy.urdf (robot description, URDF)
Before this commit: robot letter_writer_4dof, 7 links, 6 joints
Links:
- removed link cardboard
- link elbow_link: geometry visual cylinder length=0.25 radius=0.015
- link shoulder_link: geometry visual box size=0.02 0.08 0.02; visual box size=0.2 0.02 0.02
Joints:
- removed joint cardboard_fixed
- joint elbow_joint: origin xyz=0.12 0.08 0 rpy=1.5708 0 0 -> xyz=0.2 0.08 0 rpy=1.5708 0 0
- joint shoulder_extend_joint: limit lower=0.0 upper=0.25 effort=50.0 velocity=0.5 -> lower=0.0 upper=0.5 effort=50.0 velocity=0.5
- joint wrist_joint: origin xyz=0.20 0 0 rpy=0 0 0 -> xyz=0.25 0 0 rpy=0 0 0
