Commit message: Add pen retraction within letters and color-coded trajectory visualization
Updates:
- Support for pen retractions within multi-stroke letters using None markers
- Letter 'E' now draws in three separate strokes with retractions
- Added HEART shape and additional letter definitions (G, Z, M, C, D, F, J, K, O, P, Q, S, V, W, X, Y)
- Parse "HEART" as special token in letter strings
- Color-coded visualization: red for letter strokes, green for retractions/travel
- Increased animation speed (2x faster)
- Added world link to URDF for proper base rotation reference
- Improved robot geometry with updated dimensions and joint limits
- Center letters on cardboard automatically based on total letter count
- UTF-8 encoding for config file reading

File: config/robot.urdf (robot description, URDF)
Before this commit: robot letter_writer_4dof, 7 links, 6 joints
Links:
- added link world
- link elbow_link: geometry visual cylinder length=0.10 radius=0.0125; visual sphere radius=0.0125
- link shoulder_link: geometry visual cylinder length=0.03 radius=0.0125; visual cylinder length=0.22 radius=0.0125
Joints:
- added joint world_to_base_joint: type revolute, parent world, child base_link, origin xyz=0 0 0 rpy=0 0 1.5708, axis 0 0 1, limit lower=-1.5708 upper=1.5708 effort=100.0 velocity=2.0
- joint base_joint: axis 0 0 1 -> 0 1 0; limit lower=-3.14 upper=3.14 effort=100.0 velocity=2.0 -> lower=-1.57 upper=1.57 effort=100.0 velocity=2.0
- joint cardboard_fixed: parent base_link -> world
- joint elbow_joint: origin xyz=0.12 0.08 0 rpy=1.5708 0 0 -> xyz=0.22 0.03 0 rpy=1.5708 0 0
- joint shoulder_extend_joint: limit lower=0.0 upper=0.25 effort=50.0 velocity=0.5 -> lower=0.0 upper=0.40 effort=50.0 velocity=0.5; origin xyz=0.1 0 0 rpy=0 0 0 -> xyz=0.0 0 0 rpy=0 0 0
- joint wrist_joint: limit lower=-2.09 upper=0.35 effort=20.0 velocity=2.0 -> lower=-1.0472 upper=0.35 effort=20.0 velocity=2.0; origin xyz=0.20 0 0 rpy=0 0 0 -> xyz=0.10 0 0 rpy=0 0 0

Commit message: Add motor specifications and hand calculations for torque requirements
- Updated robot.urdf with motor masses and material properties
  * Base motor: 10 Nm AC servo with 1:2 gear reduction (6.5 kg)
  * Shoulder motor: 5 Nm AC servo with 1:2 gear reduction (3.2 kg)
  * Prismatic: 50 N linear actuator (0.028 kg)
  * Elbow motor: 1.2 Nm NEMA 23 stepper (0.75 kg)
  * Wrist motor: 0.5 Nm NEMA 17 stepper (0.35 kg)
  * Total system mass: 13.248 kg (10.828 kg motors + 2.420 kg structure)

- Added material definitions for visual representation
  * Steel 1018 for base (density 7850 kg/m³)
  * Aluminum 6061 for shoulder (density 2700 kg/m³)
  * Carbon fiber for arm links (density 1600 kg/m³)

- Added comprehensive hand calculations document
  * Complete manual calculations for prismatic and wrist joints
  * Sample forward kinematics calculation demonstrating methodology
  * All dynamics calculations using parallel axis theorem
  * Safety factor of 1.5x applied to all motor requirements

- Added motor requirements verification script
  * Uses Robotics Toolbox Python for computational verification
  * Calculates static torques via gravload() across multiple configurations
  * Computes dynamic torques using parallel axis theorem
  * Validates motor selections against calculated requirements

File: config/robot.urdf (robot description, URDF)
Before this commit: robot letter_writer_4dof, 8 links, 7 joints
Links:
- link base_link: mass 4.0 -> 8.405
- link elbow_link: mass 1.8 -> 0.395
- link end_effector: mass 0.07 -> 0.011
- link shoulder_base_link: mass 1.5 -> 3.348
- link shoulder_link: mass 2.0 -> 1.058
- link wrist_link: mass 1.0 -> 0.031
